Commit message: 添加了机器人末端执行器三维模型已优化moveit使用效果

File: ur5_table/urdf/ur5table2.xacro (robot description, xacro)
@@ -2,4 +2,5 @@
 <robot name="ur5table" xmlns:xacro="http://ros.org/wiki/xacro">
   <xacro:include filename="$(find ur_description)/urdf/ur5.urdf.xacro" />
+  <xacro:include filename="$(find realsense2_description)/urdf/_d435.urdf.xacro" />
   <material name="blue"><!--blue-->
     <color rgba="0.0 0.0 0.8 1.0"/>
@@ -52,3 +53,34 @@
     <origin xyz="0 0 0" rpy="0 0 3.1415926535897932346"/>
   </joint>
+  <link name="end_effector">
+    <visual>
+      <origin
+        xyz="-0.045 0 -0.085"
+        rpy="0 0 0" />
+      <geometry>
+        <mesh
+          filename="package://ur5_table/meshes/tool.STL" scale="0.001 0.001 0.001"/>
+      </geometry>
+      <material
+        name="orange">
+      </material>
+    </visual>
+    <collision>
+      <origin
+         xyz="-0.045 0 -0.085"
+        rpy="0 0 0" />
+      <geometry>
+        <mesh
+          filename="package://ur5_table/meshes/tool.STL" scale="0.001 0.001 0.001"/>
+      </geometry>
+    </collision>
+  </link>
+  <joint name="tool_to_effector" type="fixed">
+    <parent link="tool0"/>
+    <child link="end_effector"/>
+    <origin xyz="0 0 0" rpy="1.5708 0 0"/>
+  </joint>
+    <xacro:sensor_d435 parent="end_effector" name="camera">
+        <origin xyz="0 0.048 -0.085" rpy="0 0 1.5708"/>
+    </xacro:sensor_d435>
 </robot>

Commit message: 修改了TCP相对于机器人末端的姿态，并在实际机器人上进行了测试

File: ur5_table/urdf/ur5table2.xacro (robot description, xacro)
@@ -79,5 +79,5 @@
     <parent link="tool0"/>
     <child link="end_effector"/>
-    <origin xyz="0 0 0" rpy="1.5708 0 0"/>
+    <origin xyz="0 0 0" rpy="1.5708 0 -1.5708"/>
   </joint>
     <xacro:sensor_d435 parent="end_effector" name="camera">

Commit message: 添加视觉伺服位姿

File: ur5_table/urdf/ur5table2.xacro (robot description, xacro)
@@ -81,6 +81,12 @@
     <origin xyz="0 0 0" rpy="1.5708 0 -1.5708"/>
   </joint>
-    <xacro:sensor_d435 parent="end_effector" name="camera">
-        <origin xyz="0 0.048 -0.085" rpy="0 0 1.5708"/>
-    </xacro:sensor_d435>
+  <xacro:sensor_d435 parent="end_effector" name="realsense_camera">
+      <origin xyz="0 0.048 -0.085" rpy="0 0 1.5708"/>
+  </xacro:sensor_d435>
+  <link name="contact_frame"/>
+  <joint name="contact_fixed_joint" type="fixed">
+    <parent link="tool0"/>
+    <child link="contact_frame"/>
+    <origin xyz="0 0 0.122" rpy="0 0 0"/>
+  </joint>
 </robot>
